Commit message: whitespace changes.

File: kuka_lwr/lwr_description/model/kuka_lwr.gazebo.xacro (robot description, xacro)
@@ -1,39 +1,39 @@
 <?xml version="1.0"?>
 <robot xmlns:xacro="http://ros.org/wiki/xacro">
-	<xacro:macro name="kuka_lwr_gazebo" params="name">
-		<gazebo>
-			<plugin name="${name}_lwr_hw_sim" filename="liblwr_hw_gazebo_plugin.so">
-				<robotNamespace>${name}</robotNamespace>
-			</plugin>
-		</gazebo>
-		<!--gazebo>
-  			<plugin name="gazebo_ros_control" filename="libgazebo_ros_control.so">
-   			 	<robotNamespace>${name}</robotNamespace>
- 		 	</plugin>
-		</gazebo-->
-		<gazebo reference="${name}_base_link">
-			<gravity>true</gravity>
-		</gazebo>
-		<gazebo reference="${name}_1_link">
-			<gravity>true</gravity>
-		</gazebo>
-		<gazebo reference="${name}_2_link">
-			<gravity>true</gravity>
-		</gazebo>
-		<gazebo reference="${name}_3_link">
-			<gravity>true</gravity>
-		</gazebo>
-		<gazebo reference="${name}_4_link">
-			<gravity>true</gravity>
-		</gazebo>
-		<gazebo reference="${name}_5_link">
-			<gravity>true</gravity>
-		</gazebo>
-		<gazebo reference="${name}_6_link">
-			<gravity>true</gravity>
-		</gazebo>
-		<gazebo reference="${name}_7_link">
-			<gravity>true</gravity>
-		</gazebo>
-	</xacro:macro>
+  <xacro:macro name="kuka_lwr_gazebo" params="name">
+    <gazebo>
+      <plugin name="${name}_lwr_hw_sim" filename="liblwr_hw_gazebo_plugin.so">
+	<robotNamespace>${name}</robotNamespace>
+      </plugin>
+    </gazebo>
+    <!--gazebo>
+  	<plugin name="gazebo_ros_control" filename="libgazebo_ros_control.so">
+   	<robotNamespace>${name}</robotNamespace>
+ 	</plugin>
+	</gazebo-->
+    <gazebo reference="${name}_base_link">
+      <gravity>true</gravity>
+    </gazebo>
+    <gazebo reference="${name}_1_link">
+      <gravity>true</gravity>
+    </gazebo>
+    <gazebo reference="${name}_2_link">
+      <gravity>true</gravity>
+    </gazebo>
+    <gazebo reference="${name}_3_link">
+      <gravity>true</gravity>
+    </gazebo>
+    <gazebo reference="${name}_4_link">
+      <gravity>true</gravity>
+    </gazebo>
+    <gazebo reference="${name}_5_link">
+      <gravity>true</gravity>
+    </gazebo>
+    <gazebo reference="${name}_6_link">
+      <gravity>true</gravity>
+    </gazebo>
+    <gazebo reference="${name}_7_link">
+      <gravity>true</gravity>
+    </gazebo>
+  </xacro:macro>
 </robot>

File: kuka_lwr/lwr_description/model/kuka_lwr.transmission.xacro (robot description, xacro)
@@ -1,77 +1,77 @@
 <?xml version="1.0"?>
 <robot xmlns:xacro="http://ros.org/wiki/xacro">
-	<xacro:property name="Interface10" value="PositionJointInterface"/>
-	<xacro:property name="Interface30" value="EffortJointInterface"/>
-	<xacro:macro name="kuka_lwr_transmission" params="name">
-		<transmission name="${name}_0_trans">
-			<type>transmission_interface/SimpleTransmission</type>
-			<joint name="${name}_0_joint">
-				<hardwareInterface>${Interface10}</hardwareInterface>
-				<hardwareInterface>${Interface30}</hardwareInterface>
-			</joint>
-			<actuator name="${name}_0_motor">
-				<mechanicalReduction>1</mechanicalReduction>
-			</actuator>
-		</transmission>
-		<transmission name="${name}_1_trans">
-			<type>transmission_interface/SimpleTransmission</type>
-			<joint name="${name}_1_joint">
-				<hardwareInterface>${Interface10}</hardwareInterface>
-				<hardwareInterface>${Interface30}</hardwareInterface>
-			</joint>
-			<actuator name="${name}_1_motor">
-				<mechanicalReduction>1</mechanicalReduction>
-			</actuator>
-		</transmission>
-		<transmission name="${name}_2_trans">
-			<type>transmission_interface/SimpleTransmission</type>
-			<joint name="${name}_2_joint">
-				<hardwareInterface>${Interface10}</hardwareInterface>
-				<hardwareInterface>${Interface30}</hardwareInterface>
-			</joint>
-			<actuator name="${name}_2_motor">
-				<mechanicalReduction>1</mechanicalReduction>
-			</actuator>
-		</transmission>
-		<transmission name="${name}_3_trans">
-			<type>transmission_interface/SimpleTransmission</type>
-			<joint name="${name}_3_joint">
-				<hardwareInterface>${Interface10}</hardwareInterface>
-				<hardwareInterface>${Interface30}</hardwareInterface>
-			</joint>
-			<actuator name="${name}_3_motor">
-				<mechanicalReduction>1</mechanicalReduction>
-			</actuator>
-		</transmission>
-		<transmission name="${name}_4_trans">
-			<type>transmission_interface/SimpleTransmission</type>
-			<joint name="${name}_4_joint">
-				<hardwareInterface>${Interface10}</hardwareInterface>
-				<hardwareInterface>${Interface30}</hardwareInterface>
-			</joint>
-			<actuator name="${name}_4_motor">
-				<mechanicalReduction>1</mechanicalReduction>
-			</actuator>
-		</transmission>
-		<transmission name="${name}_5_trans">
-			<type>transmission_interface/SimpleTransmission</type>
-			<joint name="${name}_5_joint">
-				<hardwareInterface>${Interface10}</hardwareInterface>
-				<hardwareInterface>${Interface30}</hardwareInterface>
-			</joint>
-			<actuator name="${name}_5_motor">
-				<mechanicalReduction>1</mechanicalReduction>
-			</actuator>
-		</transmission>
-		<transmission name="${name}_6_trans">
-			<type>transmission_interface/SimpleTransmission</type>
-			<joint name="${name}_6_joint">
-				<hardwareInterface>${Interface10}</hardwareInterface>
-				<hardwareInterface>${Interface30}</hardwareInterface>
-			</joint>
-			<actuator name="${name}_6_motor">
-				<mechanicalReduction>1</mechanicalReduction>
-			</actuator>
-		</transmission>
-	</xacro:macro>
+  <xacro:property name="Interface10" value="PositionJointInterface"/>
+  <xacro:property name="Interface30" value="EffortJointInterface"/>
+  <xacro:macro name="kuka_lwr_transmission" params="name">
+    <transmission name="${name}_0_trans">
+      <type>transmission_interface/SimpleTransmission</type>
+      <joint name="${name}_0_joint">
+	<hardwareInterface>${Interface10}</hardwareInterface>
+	<hardwareInterface>${Interface30}</hardwareInterface>
+      </joint>
+      <actuator name="${name}_0_motor">
+	<mechanicalReduction>1</mechanicalReduction>
+      </actuator>
+    </transmission>
+    <transmission name="${name}_1_trans">
+      <type>transmission_interface/SimpleTransmission</type>
+      <joint name="${name}_1_joint">
+	<hardwareInterface>${Interface10}</hardwareInterface>
+	<hardwareInterface>${Interface30}</hardwareInterface>
+      </joint>
+      <actuator name="${name}_1_motor">
+	<mechanicalReduction>1</mechanicalReduction>
+      </actuator>
+    </transmission>
+    <transmission name="${name}_2_trans">
+      <type>transmission_interface/SimpleTransmission</type>
+      <joint name="${name}_2_joint">
+	<hardwareInterface>${Interface10}</hardwareInterface>
+	<hardwareInterface>${Interface30}</hardwareInterface>
+      </joint>
+      <actuator name="${name}_2_motor">
+	<mechanicalReduction>1</mechanicalReduction>
+      </actuator>
+    </transmission>
+    <transmission name="${name}_3_trans">
+      <type>transmission_interface/SimpleTransmission</type>
+      <joint name="${name}_3_joint">
+	<hardwareInterface>${Interface10}</hardwareInterface>
+	<hardwareInterface>${Interface30}</hardwareInterface>
+      </joint>
+      <actuator name="${name}_3_motor">
+	<mechanicalReduction>1</mechanicalReduction>
+      </actuator>
+    </transmission>
+    <transmission name="${name}_4_trans">
+      <type>transmission_interface/SimpleTransmission</type>
+      <joint name="${name}_4_joint">
+	<hardwareInterface>${Interface10}</hardwareInterface>
+	<hardwareInterface>${Interface30}</hardwareInterface>
+      </joint>
+      <actuator name="${name}_4_motor">
+	<mechanicalReduction>1</mechanicalReduction>
+      </actuator>
+    </transmission>
+    <transmission name="${name}_5_trans">
+      <type>transmission_interface/SimpleTransmission</type>
+      <joint name="${name}_5_joint">
+	<hardwareInterface>${Interface10}</hardwareInterface>
+	<hardwareInterface>${Interface30}</hardwareInterface>
+      </joint>
+      <actuator name="${name}_5_motor">
+	<mechanicalReduction>1</mechanicalReduction>
+      </actuator>
+    </transmission>
+    <transmission name="${name}_6_trans">
+      <type>transmission_interface/SimpleTransmission</type>
+      <joint name="${name}_6_joint">
+	<hardwareInterface>${Interface10}</hardwareInterface>
+	<hardwareInterface>${Interface30}</hardwareInterface>
+      </joint>
+      <actuator name="${name}_6_motor">
+	<mechanicalReduction>1</mechanicalReduction>
+      </actuator>
+    </transmission>
+  </xacro:macro>
 </robot>
