Commit message: whitespace changes.

File: kuka_lwr/lwr_description/model/kuka_lwr.urdf.xacro (robot description, xacro)
@@ -1,495 +1,495 @@
 <?xml version="1.0"?>
 <robot name="kuka_lwr" xmlns:xacro="http://www.ros.org/wiki/xacro">
-	<!-- utils /-->
-	<xacro:include filename="$(find lwr_description)/model/utils.xacro"/>
-	<xacro:include filename="$(find lwr_description)/model/kuka_materials.xacro"
-	/>
-	<!-- gazebo and transmission models /-->
-	<xacro:include filename="$(find lwr_description)/model/kuka_lwr.gazebo.xacro"/>
-	<xacro:include filename="$(find lwr_description)/model/kuka_lwr.transmission.xacro"/>
-	<!-- properties /-->
-	<xacro:property name="base_mass" value="2.0"/>
-	<xacro:property name="link_mass" value="2.0"/>
-	<xacro:property name="velocity_scale" value="1"/>
-	<xacro:property name="effort_scale" value="1"/>
-	<xacro:property name="max_stiffness" value="5000"/>
-	<xacro:property name="min_stiffness" value="0"/>
-	<xacro:property name="rate_stiffness" value="20000"/> <!-- reflex to stiffness -->
-	<xacro:property name="max_damping" value="500"/>
-	<xacro:property name="min_damping" value="0"/>
-	<xacro:property name="rate_daming" value="20000"/>
-	<!-- URDF model /-->
-	<xacro:macro name="kuka_lwr" params="name *origin">
-	<link name="world"/>
-	<gazebo reference="world">
-    		<static>true</static>
-    		<turnGravityOff>true</turnGravityOff>
-	</gazebo>
-		<!-- First (shoulder) element of the arm. Fixed to its parent. -->
-		<joint name="${name}_base_joint" type="fixed">
-			<insert_block name="origin"/>
-			<origin xyz="0 0 0" rpy="0 0 0"/>
-			<parent link="world"/>
-			<child link="${name}_base_link"/>
-		</joint>
-		<link name="${name}_base_link">
-			<inertial>
-				<mass value="${base_mass}"/>
-				<origin xyz="0 0 0.055"  />
-				<cylinder_inertia_def radius="0.06" length="0.11" mass="${base_mass}"/>
-			</inertial>
-			<visual>
-				<origin xyz="0 0 0" rpy="0 0 ${M_PI}"/>
-				<geometry>
-					<mesh filename="package://lwr_description/meshes/base.dae"/>
-				</geometry>
-				<material name="Kuka/Orange"/>
-			</visual>
-			<collision>
-				<origin xyz="0 0 0.055" rpy="0 0 ${M_PI}"/>
-				<geometry>
-					<!-- <mesh filename="package://lwr_description/meshes/convex/arm_base_convex.stl"/> -->
-					<cylinder radius="0.07" length="0.11"/>
-				</geometry>
-			</collision>
-		</link>
-		<!-- Second segment of the arm. Joint along z-axis -->
-		<joint name="${name}_0_joint" type="revolute">
-			<origin xyz="0 0 0.11" rpy="0 0 0"/>
-			<axis xyz="0 0 1"/>
-			<limit lower="${-170 * M_PI / 180}" upper="${170 * M_PI / 180}" effort="176" velocity="${velocity_scale * 110 * M_PI / 180}" />
-			<dynamics friction="10.0" damping="1.0"/>
-			<parent link="${name}_base_link"/>
-			<child link="${name}_1_link"/>
-		</joint>
-		<joint name="${name}_0_joint_stiffness" type="revolute">
-			<axis xyz="0 0 1"/>
-			<limit lower="${min_stiffness}" upper="${max_stiffness}" effort="0" velocity="${rate_stiffness}" />
-			<safety_controller soft_lower_limit="${min_stiffness}" soft_upper_limit="${max_stiffness}" k_position="30" k_velocity="30"/>
-			<parent link="${name}_base_link"/>
-			<child link="${name}_1_link_dummy"/>
-		</joint>
-		<joint name="${name}_0_joint_damping" type="revolute">
-			<axis xyz="0 0 1"/>
-			<limit lower="${min_damping}" upper="${max_damping}" effort="0" velocity="${rate_daming}" />
-			<safety_controller soft_lower_limit="${min_damping}" soft_upper_limit="${max_damping}" k_position="30" k_velocity="30"/>
-			<parent link="${name}_base_link"/>
-			<child link="${name}_1_link_damping"/>
-		</joint>
-		<joint name="${name}_0_joint_torque" type="revolute">
-			<axis xyz="0 0 1"/>
-			<limit lower="${-170 * M_PI / 180}" upper="${170 * M_PI / 180}" effort="176" velocity="${velocity_scale * 110 * M_PI / 180}" />
-			<dynamics friction="10.0" damping="1.0"/>
-			<parent link="${name}_base_link"/>
-			<child link="${name}_1_link_torque"/>
-		</joint>
-		<link name="${name}_1_link_dummy"/>
-		<link name="${name}_1_link_damping"/>
-		<link name="${name}_1_link_torque"/>
-		<link name="${name}_1_link">
-			<inertial>
-				<mass value="${link_mass}"/>
-				<origin rpy="0 0 0" xyz="0 -0.06 0.130"/>
-				<cuboid_inertia_def length="0.12" width="0.06" height="0.260" mass="${link_mass}"/>
-			</inertial>
-			<visual>
-				<origin xyz="0 0 -0.008" rpy="0 0 ${M_PI}"/>
-				<geometry>
-					<mesh filename="package://lwr_description/meshes/link_1.dae"/>
-				</geometry>
-				<material name="Kuka/Orange"/>
-			</visual>
-			<collision>
-				<origin xyz="0 0 0.0" rpy="0 0 0"/>
-				<geometry>
-					<!--mesh filename="package://lwr_description/meshes/convex/arm_segment_a_convex.stl"/-->
-					<sphere radius="0.07"/>
-				</geometry>
-			</collision>
-			<collision>
-				<origin xyz="0 0.06 0.2" rpy="0 0 0"/>
-				<geometry>
-					<sphere radius="0.07"/>
-				</geometry>
-			</collision>
-			<collision>
-				<origin xyz="0 0.03 0.1" rpy="-0.291 0 0"/>
-				<geometry>
-					<cylinder radius="0.07" length="0.208"/>
-				</geometry>
-			</collision>
-		</link>
-		<!-- Third segment of the arm. Joint along y-axis -->
-		<joint name="${name}_1_joint" type="revolute">
-			<origin xyz="0 0 0.2005" rpy="0 0 0"/>
-			<axis xyz="0 -1 0"/>
-			<limit lower="${-120 * M_PI / 180}" upper="${120 * M_PI / 180}" effort="176" velocity="${velocity_scale * 110 * M_PI / 180}" />
-			<dynamics friction="10.0" damping="1.0"/>
-			<parent link="${name}_1_link"/>
-			<child link="${name}_2_link"/>
-		</joint>
-		<joint name="${name}_1_joint_stiffness" type="revolute">
-			<axis xyz="0 0 1"/>
-			<limit lower="${min_stiffness}" upper="${max_stiffness}" effort="0" velocity="${rate_stiffness}" />
-			<safety_controller soft_lower_limit="${min_stiffness}" soft_upper_limit="${max_stiffness}" k_position="30" k_velocity="30"/>
-			<parent link="${name}_1_link"/>
-			<child link="${name}_2_link_dummy"/>
-		</joint>
-		<joint name="${name}_1_joint_damping" type="revolute">
-			<axis xyz="0 0 1"/>
-			<limit lower="${min_damping}" upper="${max_damping}" effort="0" velocity="${rate_daming}" />
-			<safety_controller soft_lower_limit="${min_damping}" soft_upper_limit="${max_damping}" k_position="30" k_velocity="30"/>
-			<parent link="${name}_1_link"/>
-			<child link="${name}_2_link_damping"/>
-		</joint>
-		<joint name="${name}_1_joint_torque" type="revolute">
-			<axis xyz="0 -1 0"/>
-			<limit lower="${-120 * M_PI / 180}" upper="${120 * M_PI / 180}" effort="176" velocity="${velocity_scale * 110 * M_PI / 180}" />
-			<dynamics friction="10.0" damping="1.0"/>
-			<parent link="${name}_1_link"/>
-			<child link="${name}_2_link_torque"/>
-		</joint>
-		<link name="${name}_2_link_dummy"/>
-		<link name="${name}_2_link_damping"/>
-		<link name="${name}_2_link_torque"/>
-		<link name="${name}_2_link">
-			<inertial>
-				<mass value="${link_mass}"/>
-				<origin rpy="0 0 0" xyz="0 0.06 ${0.130 - 0.06}"/>
-				<cuboid_inertia_def length="0.12" width="0.06" height="0.260" mass="${link_mass}"/>
-			</inertial>
-			<visual>
-				<origin xyz="0 0 0.0" rpy="0 0 ${M_PI}"/>
-				<geometry>
-					<mesh filename="package://lwr_description/meshes/link_2.dae"/>
-				</geometry>
-				<!--material name="Kuka/Orange"/-->
-			</visual>
-			<collision>
-				<origin xyz="0 0 0.2" rpy="0 0 0"/>
-				<geometry>
-					<!--mesh filename="package://lwr_description/meshes/convex/arm_segment_b_convex.stl"/-->
-					<sphere radius="0.07"/>
-				</geometry>
-			</collision>
-			<collision>
-				<origin xyz="0 -0.06 0.0" rpy="0 0 0"/>
-				<geometry>
-					<sphere radius="0.07"/>
-				</geometry>
-			</collision>
-			<collision>
-				<origin xyz="0 -0.03 0.1" rpy="-0.291 0 0"/>
-				<geometry>
-					<cylinder radius="0.07" length="0.208"/>
-				</geometry>
-			</collision>
-		</link>
-		<!-- Fourth element of the arm. z-axis -->
-		<joint name="${name}_2_joint" type="revolute">
-			<origin xyz="0 0 0.20" rpy="0 0 0"/>
-			<axis xyz="0 0 1"/>
-			<limit lower="${-170 * M_PI / 180}" upper="${170 * M_PI / 180}" effort="100" velocity="${velocity_scale * 128 * M_PI / 180}" />
-			<dynamics friction="10.0" damping="1.0"/>
-			<parent link="${name}_2_link"/>
-			<child link="${name}_3_link"/>
-		</joint>
-		<joint name="${name}_2_joint_stiffness" type="revolute">
-			<axis xyz="0 0 1"/>
-			<limit lower="${min_stiffness}" upper="${max_stiffness}" effort="0" velocity="${rate_stiffness}" />
-			<safety_controller soft_lower_limit="${min_stiffness}" soft_upper_limit="${max_stiffness}" k_position="30" k_velocity="30"/>
-			<parent link="${name}_2_link"/>
-			<child link="${name}_3_link_dummy"/>
-		</joint>
-		<joint name="${name}_2_joint_damping" type="revolute">
-			<axis xyz="0 0 1"/>
-			<limit lower="${min_damping}" upper="${max_damping}" effort="0" velocity="${rate_daming}" />
-			<safety_controller soft_lower_limit="${min_damping}" soft_upper_limit="${max_damping}" k_position="30" k_velocity="30"/>
-			<parent link="${name}_2_link"/>
-			<child link="${name}_3_link_damping"/>
-		</joint>
-		<joint name="${name}_2_joint_torque" type="revolute">
-			<axis xyz="0 0 1"/>
-			<limit lower="${min_stiffness}" upper="${max_stiffness}" effort="0" velocity="${rate_stiffness}" />
-			<safety_controller soft_lower_limit="${min_stiffness}" soft_upper_limit="${max_stiffness}" k_position="30" k_velocity="30"/>
-			<parent link="${name}_2_link"/>
-			<child link="${name}_3_link_torque"/>
-		</joint>
-		<link name="${name}_3_link_dummy"/>
-		<link name="${name}_3_link_damping"/>
-		<link name="${name}_3_link_torque"/>
-		<link name="${name}_3_link">
-			<inertial>
-				<mass value="${link_mass}"/>
-				<origin rpy="0 0 0" xyz="0 0.06 0.130"/>
-				<cuboid_inertia_def length="0.12" width="0.06" height="0.260" mass="${link_mass}"/>
-			</inertial>
-			<visual>
-				<origin xyz="0 0 -0.008" rpy="0 0 ${M_PI}"/>
-				<geometry>
-					<mesh filename="package://lwr_description/meshes/link_3.dae"/>
-				</geometry>
-				<material name="Kuka/Orange"/>
-			</visual>
-			<collision>
-				<origin xyz="0 0 0.0" rpy="0 0 0"/>
-				<geometry>
-					<!--mesh filename="package://lwr_description/meshes/convex/arm_segment_a_convex.stl"/-->
-					<sphere radius="0.07"/>
-				</geometry>
-			</collision>
-			<collision>
-				<origin xyz="0 -0.06 0.2" rpy="0 0 0"/>
-				<geometry>
-					<sphere radius="0.07"/>
-				</geometry>
-			</collision>
-			<collision>
-				<origin xyz="0 -0.03 0.1" rpy="0.291 0 0"/>
-				<geometry>
-					<cylinder radius="0.07" length="0.208"/>
-				</geometry>
-			</collision>
-		</link>
-		<!-- fifth element of the arm. x-axis -->
-		<joint name="${name}_3_joint" type="revolute">
-			<origin xyz="0 0 0.20" rpy="0 0 0"/>
-			<axis xyz="0 1 0"/>
-			<limit lower="${-120 * M_PI / 180}" upper="${120 * M_PI / 180}" effort="100" velocity="${velocity_scale * 128 * M_PI / 180}" />
-			<dynamics friction="10.0" damping="1.0"/>
-			<parent link="${name}_3_link"/>
-			<child link="${name}_4_link"/>
-		</joint>
-		<joint name="${name}_3_joint_stiffness" type="revolute">
-			<axis xyz="0 0 1"/>
-			<limit lower="${min_stiffness}" upper="${max_stiffness}" effort="0" velocity="${rate_stiffness}" />
-			<safety_controller soft_lower_limit="${min_stiffness}" soft_upper_limit="${max_stiffness}" k_position="30" k_velocity="30"/>
-			<parent link="${name}_3_link"/>
-			<child link="${name}_4_link_dummy"/>
-		</joint>
-		<joint name="${name}_3_joint_damping" type="revolute">
-			<axis xyz="0 0 1"/>
-			<limit lower="${min_damping}" upper="${max_damping}" effort="0" velocity="${rate_daming}" />
-			<safety_controller soft_lower_limit="${min_damping}" soft_upper_limit="${max_damping}" k_position="30" k_velocity="30"/>
-			<parent link="${name}_3_link"/>
-			<child link="${name}_4_link_damping"/>
-		</joint>
-		<joint name="${name}_3_joint_torque" type="revolute">
-			<axis xyz="0 1 0"/>
-			<limit lower="${-120 * M_PI / 180}" upper="${120 * M_PI / 180}" effort="100" velocity="${velocity_scale * 128 * M_PI / 180}" />
-			<dynamics friction="10.0" damping="1.0"/>
-			<parent link="${name}_3_link"/>
-			<child link="${name}_4_link_torque"/>
-		</joint>
-		<link name="${name}_4_link_dummy"/>
-		<link name="${name}_4_link_damping"/>
-		<link name="${name}_4_link_torque"/>
-		<link name="${name}_4_link">
-			<inertial>
-				<mass value="${link_mass}"/>
-				<origin rpy="0 0 0" xyz="0 -0.06 ${0.130 - 0.06}"/>
-				<cuboid_inertia_def length="0.12" width="0.06" height="0.2600" mass="${link_mass}"/>
-			</inertial>
-			<visual>
-				<origin xyz="0 0 0.0" rpy="0 0 ${M_PI}"/>
-				<geometry>
-					<mesh filename="package://lwr_description/meshes/link_4.dae"/>
-				</geometry>
-				<material name="Kuka/Orange"/>
-			</visual>
-			<collision>
-			<origin xyz="0 0 0.2" rpy="0 0 0"/>
-			<geometry>
-				<!--mesh filename="package://lwr_description/meshes/convex/arm_segment_b_convex.stl"/-->
-				<sphere radius="0.07"/>
-			</geometry>
-			</collision>
-			<collision>
-				<origin xyz="0 0.06 0.0" rpy="0 0 0"/>
-				<geometry>
-					<sphere radius="0.07"/>
-				</geometry>
-			</collision>
-			<collision>
-				<origin xyz="0 0.03 0.1" rpy="0.291 0 0"/>
-				<geometry>
-					<cylinder radius="0.07" length="0.208"/>
-				</geometry>
-			</collision>
-		</link>
-		<!-- Sixth element of the arm. z-axis -->
-		<joint name="${name}_4_joint" type="revolute">
-			<origin xyz="0 0 0.20" rpy="0 0 0"/>
-			<axis xyz="0 0 1"/>
-			<limit lower="${-170 * M_PI / 180}" upper="${170 * M_PI / 180}" effort="100" velocity="${velocity_scale * 204 * M_PI / 180}" />
-			<dynamics friction="10.0" damping="1.0"/>
-			<parent link="${name}_4_link"/>
-			<child link="${name}_5_link"/>
-		</joint>
-		<joint name="${name}_4_joint_stiffness" type="revolute">
-			<axis xyz="0 0 1"/>
-			<limit lower="${min_stiffness}" upper="${max_stiffness}" effort="0" velocity="${rate_stiffness}" />
-			<safety_controller soft_lower_limit="${min_stiffness}" soft_upper_limit="${max_stiffness}" k_position="30" k_velocity="30"/>
-			<parent link="${name}_4_link"/>
-			<child link="${name}_5_link_dummy"/>
-		</joint>
-		<joint name="${name}_4_joint_damping" type="revolute">
-			<axis xyz="0 0 1"/>
-			<limit lower="${min_damping}" upper="${max_damping}" effort="0" velocity="${rate_daming}" />
-			<safety_controller soft_lower_limit="${min_damping}" soft_upper_limit="${max_damping}" k_position="30" k_velocity="30"/>
-			<parent link="${name}_4_link"/>
-			<child link="${name}_5_link_damping"/>
-		</joint>
-		<joint name="${name}_4_joint_torque" type="revolute">
-			<axis xyz="0 0 1"/>
-			<limit lower="${min_damping}" upper="${max_damping}" effort="0" velocity="${rate_daming}" />
-			<safety_controller soft_lower_limit="${min_damping}" soft_upper_limit="${max_damping}" k_position="30" k_velocity="30"/>
-			<parent link="${name}_4_link"/>
-			<child link="${name}_5_link_torque"/>
-		</joint>
-		<link name="${name}_5_link_dummy"/>
-		<link name="${name}_5_link_damping"/>
-		<link name="${name}_5_link_torque"/>
-		<link name="${name}_5_link">
-			<inertial>
-				<mass value="${link_mass}"/>
-				<origin rpy="0 0 0" xyz="0 0 0.124"/>
-				<cuboid_inertia_def length="0.12" width="0.06" height="0.248" mass="${link_mass}"/>
-			</inertial>
-			<visual>
-				<origin xyz="0 0 -0.008" rpy="0 0 ${M_PI}"/>
-				<geometry name="${name}_5_geom">
-					<mesh filename="package://lwr_description/meshes/link_5.dae"/>
-				</geometry>
-				<material name="Kuka/Orange"/>
-			</visual>
-			<collision>
-				<origin xyz="0 0 0.0" rpy="0 0 0"/>
-				<geometry>
-					<!--mesh filename="package://lwr_description/meshes/convex/arm_segment_last_convex.stl"/-->
-					<sphere radius="0.07"/>
-				</geometry>
-			</collision>
-			<collision>
-				<origin xyz="0 0.04 0.19" rpy="0 0 0"/>
-				<geometry>
-					<sphere radius="0.07"/>
-				</geometry>
-			</collision>
-			<collision>
-				<origin xyz="0 0.02 0.095" rpy="-0.207 0 0"/>
-				<geometry>
-					<cylinder radius="0.07" length="0.198"/>
-				</geometry>
-			</collision>
-		</link>
-		<!-- Seventh element of the arm. z-axis -->
-		<joint name="${name}_5_joint" type="revolute">
-			<origin xyz="0 0 0.19" rpy="0 0 0"/>
-			<axis xyz="0 -1 0"/>
-			<limit lower="${-120 * M_PI / 180}" upper="${120 * M_PI / 180}" effort="38" velocity="${velocity_scale * 184 * M_PI / 180}" />
-			<dynamics friction="10.0" damping="1.0"/>
-			<parent link="${name}_5_link"/>
-			<child link="${name}_6_link"/>
-		</joint>
-		<joint name="${name}_5_joint_stiffness" type="revolute">
-			<axis xyz="0 0 1"/>
-			<limit lower="${min_stiffness}" upper="${max_stiffness}" effort="0" velocity="${rate_stiffness}" />
-			<safety_controller soft_lower_limit="${min_stiffness}" soft_upper_limit="${max_stiffness}" k_position="30" k_velocity="30"/>
-			<parent link="${name}_5_link"/>
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
File: kuka_lwr/single_lwr_example/single_lwr_robot/robot/single_lwr_robot.urdf.xacro (robot description, xacro)
@@ -1,9 +1,9 @@
 <?xml version="1.0"?>
 <robot xmlns:xacro="http://www.ros.org/wiki/xacro" name="single_lwr_robot">
-	<!-- Include all models -->
-	<xacro:include filename="$(find lwr_description)/model/kuka_lwr.urdf.xacro"/>
-	<!-- using the models -->
-	<xacro:kuka_lwr name="lwr">
-		<origin xyz="0 0 0" rpy="0 0 0"/>
-	</xacro:kuka_lwr>
+  <!-- Include all models -->
+  <xacro:include filename="$(find lwr_description)/model/kuka_lwr.urdf.xacro"/>
+  <!-- using the models -->
+  <xacro:kuka_lwr name="lwr">
+    <origin xyz="0 0 0" rpy="0 0 0"/>
+  </xacro:kuka_lwr>
 </robot>
