Commit message: .

File: kuka_lwr/lwr_description/model/kuka_lwr.urdf.xacro (robot description, xacro)
@@ -16,4 +16,7 @@
 	<xacro:property name="min_stiffness" value="0"/>
 	<xacro:property name="rate_stiffness" value="20000"/> <!-- reflex to stiffness -->
+	<xacro:property name="max_damping" value="500"/>
+	<xacro:property name="min_damping" value="0"/>
+	<xacro:property name="rate_daming" value="20000"/>
 	<!-- URDF model /-->
 	<xacro:macro name="kuka_lwr" params="name *origin">
@@ -67,5 +70,13 @@
 			<child link="${name}_1_link_dummy"/>
 		</joint>
+		<joint name="${name}_0_joint_damping" type="revolute">
+			<axis xyz="0 0 1"/>
+			<limit lower="${min_damping}" upper="${max_damping}" effort="0" velocity="${rate_daming}" />
+			<safety_controller soft_lower_limit="${min_damping}" soft_upper_limit="${max_damping}" k_position="30" k_velocity="30"/>
+			<parent link="${name}_base_link"/>
+			<child link="${name}_1_link_damping"/>
+		</joint>
 		<link name="${name}_1_link_dummy"/>
+		<link name="${name}_1_link_damping"/>
 		<link name="${name}_1_link">
 			<inertial>
@@ -117,5 +128,13 @@
 			<child link="${name}_2_link_dummy"/>
 		</joint>
+		<joint name="${name}_1_joint_damping" type="revolute">
+			<axis xyz="0 0 1"/>
+			<limit lower="${min_damping}" upper="${max_damping}" effort="0" velocity="${rate_daming}" />
+			<safety_controller soft_lower_limit="${min_damping}" soft_upper_limit="${max_damping}" k_position="30" k_velocity="30"/>
+			<parent link="${name}_1_link"/>
+			<child link="${name}_2_link_damping"/>
+		</joint>
 		<link name="${name}_2_link_dummy"/>
+		<link name="${name}_2_link_damping"/>
 		<link name="${name}_2_link">
 			<inertial>
@@ -167,5 +186,13 @@
 			<child link="${name}_3_link_dummy"/>
 		</joint>
+		<joint name="${name}_2_joint_damping" type="revolute">
+			<axis xyz="0 0 1"/>
+			<limit lower="${min_damping}" upper="${max_damping}" effort="0" velocity="${rate_daming}" />
+			<safety_controller soft_lower_limit="${min_damping}" soft_upper_limit="${max_damping}" k_position="30" k_velocity="30"/>
+			<parent link="${name}_2_link"/>
+			<child link="${name}_3_link_damping"/>
+		</joint>
 		<link name="${name}_3_link_dummy"/>
+		<link name="${name}_3_link_damping"/>
 		<link name="${name}_3_link">
 			<inertial>
@@ -217,5 +244,13 @@
 			<child link="${name}_4_link_dummy"/>
 		</joint>
+		<joint name="${name}_3_joint_damping" type="revolute">
+			<axis xyz="0 0 1"/>
+			<limit lower="${min_damping}" upper="${max_damping}" effort="0" velocity="${rate_daming}" />
+			<safety_controller soft_lower_limit="${min_damping}" soft_upper_limit="${max_damping}" k_position="30" k_velocity="30"/>
+			<parent link="${name}_3_link"/>
+			<child link="${name}_4_link_damping"/>
+		</joint>
 		<link name="${name}_4_link_dummy"/>
+		<link name="${name}_4_link_damping"/>
 		<link name="${name}_4_link">
 			<inertial>
@@ -267,5 +302,13 @@
 			<child link="${name}_5_link_dummy"/>
 		</joint>
+		<joint name="${name}_4_joint_damping" type="revolute">
+			<axis xyz="0 0 1"/>
+			<limit lower="${min_damping}" upper="${max_damping}" effort="0" velocity="${rate_daming}" />
+			<safety_controller soft_lower_limit="${min_damping}" soft_upper_limit="${max_damping}" k_position="30" k_velocity="30"/>
+			<parent link="${name}_4_link"/>
+			<child link="${name}_5_link_damping"/>
+		</joint>
 		<link name="${name}_5_link_dummy"/>
+		<link name="${name}_5_link_damping"/>
 		<link name="${name}_5_link">
 			<inertial>
@@ -317,5 +360,13 @@
 			<child link="${name}_6_link_dummy"/>
 		</joint>
+		<joint name="${name}_5_joint_damping" type="revolute">
+			<axis xyz="0 0 1"/>
+			<limit lower="${min_damping}" upper="${max_damping}" effort="0" velocity="${rate_daming}" />
+			<safety_controller soft_lower_limit="${min_damping}" soft_upper_limit="${max_damping}" k_position="30" k_velocity="30"/>
+			<parent link="${name}_5_link"/>
+			<child link="${name}_6_link_damping"/>
+		</joint>
 		<link name="${name}_6_link_dummy"/>
+		<link name="${name}_6_link_damping"/>
 		<link name="${name}_6_link">
 			<inertial>
@@ -354,5 +405,13 @@
 			<child link="${name}_7_link_dummy"/>
 		</joint>
+		<joint name="${name}_6_joint_damping" type="revolute">
+			<axis xyz="0 0 1"/>
+			<limit lower="${min_damping}" upper="${max_damping}" effort="0" velocity="${rate_daming}" />
+			<safety_controller soft_lower_limit="${min_damping}" soft_upper_limit="${max_damping}" k_position="30" k_velocity="30"/>
+			<parent link="${name}_6_link"/>
+			<child link="${name}_7_link_damping"/>
+		</joint>
 		<link name="${name}_7_link_dummy"/>
+		<link name="${name}_7_link_damping"/>
 		<link name="${name}_7_link">
 			<inertial>

Commit message: .

File: kuka_lwr/lwr_description/model/kuka_lwr.urdf.xacro (robot description, xacro)
@@ -77,6 +77,14 @@
 			<child link="${name}_1_link_damping"/>
 		</joint>
+		<joint name="${name}_0_joint_torque" type="revolute">
+			<axis xyz="0 0 1"/>
+			<limit lower="${-170 * M_PI / 180}" upper="${170 * M_PI / 180}" effort="176" velocity="${velocity_scale * 110 * M_PI / 180}" />
+			<dynamics friction="10.0" damping="1.0"/>
+			<parent link="${name}_base_link"/>
+			<child link="${name}_1_link_torque"/>
+		</joint>
 		<link name="${name}_1_link_dummy"/>
 		<link name="${name}_1_link_damping"/>
+		<link name="${name}_1_link_torque"/>
 		<link name="${name}_1_link">
 			<inertial>
@@ -135,6 +143,14 @@
 			<child link="${name}_2_link_damping"/>
 		</joint>
+		<joint name="${name}_1_joint_torque" type="revolute">
+			<axis xyz="0 -1 0"/>
+			<limit lower="${-120 * M_PI / 180}" upper="${120 * M_PI / 180}" effort="176" velocity="${velocity_scale * 110 * M_PI / 180}" />
+			<dynamics friction="10.0" damping="1.0"/>
+			<parent link="${name}_1_link"/>
+			<child link="${name}_2_link_torque"/>
+		</joint>
 		<link name="${name}_2_link_dummy"/>
 		<link name="${name}_2_link_damping"/>
+		<link name="${name}_2_link_torque"/>
 		<link name="${name}_2_link">
 			<inertial>
@@ -193,6 +209,14 @@
 			<child link="${name}_3_link_damping"/>
 		</joint>
+		<joint name="${name}_2_joint_torque" type="revolute">
+			<axis xyz="0 0 1"/>
+			<limit lower="${min_stiffness}" upper="${max_stiffness}" effort="0" velocity="${rate_stiffness}" />
+			<safety_controller soft_lower_limit="${min_stiffness}" soft_upper_limit="${max_stiffness}" k_position="30" k_velocity="30"/>
+			<parent link="${name}_2_link"/>
+			<child link="${name}_3_link_torque"/>
+		</joint>
 		<link name="${name}_3_link_dummy"/>
 		<link name="${name}_3_link_damping"/>
+		<link name="${name}_3_link_torque"/>
 		<link name="${name}_3_link">
 			<inertial>
@@ -251,6 +275,14 @@
 			<child link="${name}_4_link_damping"/>
 		</joint>
+		<joint name="${name}_3_joint_torque" type="revolute">
+			<axis xyz="0 1 0"/>
+			<limit lower="${-120 * M_PI / 180}" upper="${120 * M_PI / 180}" effort="100" velocity="${velocity_scale * 128 * M_PI / 180}" />
+			<dynamics friction="10.0" damping="1.0"/>
+			<parent link="${name}_3_link"/>
+			<child link="${name}_4_link_torque"/>
+		</joint>
 		<link name="${name}_4_link_dummy"/>
 		<link name="${name}_4_link_damping"/>
+		<link name="${name}_4_link_torque"/>
 		<link name="${name}_4_link">
 			<inertial>
@@ -309,6 +341,14 @@
 			<child link="${name}_5_link_damping"/>
 		</joint>
+		<joint name="${name}_4_joint_torque" type="revolute">
+			<axis xyz="0 0 1"/>
+			<limit lower="${min_damping}" upper="${max_damping}" effort="0" velocity="${rate_daming}" />
+			<safety_controller soft_lower_limit="${min_damping}" soft_upper_limit="${max_damping}" k_position="30" k_velocity="30"/>
+			<parent link="${name}_4_link"/>
+			<child link="${name}_5_link_torque"/>
+		</joint>
 		<link name="${name}_5_link_dummy"/>
 		<link name="${name}_5_link_damping"/>
+		<link name="${name}_5_link_torque"/>
 		<link name="${name}_5_link">
 			<inertial>
@@ -367,6 +407,14 @@
 			<child link="${name}_6_link_damping"/>
 		</joint>
+		<joint name="${name}_5_joint_torque" type="revolute">
+			<axis xyz="0 0 1"/>
+			<limit lower="${min_damping}" upper="${max_damping}" effort="0" velocity="${rate_daming}" />
+			<safety_controller soft_lower_limit="${min_damping}" soft_upper_limit="${max_damping}" k_position="30" k_velocity="30"/>
+			<parent link="${name}_5_link"/>
+			<child link="${name}_6_link_torque"/>
+		</joint>
 		<link name="${name}_6_link_dummy"/>
 		<link name="${name}_6_link_damping"/>
+		<link name="${name}_6_link_torque"/>
 		<link name="${name}_6_link">
 			<inertial>
@@ -412,6 +460,14 @@
 			<child link="${name}_7_link_damping"/>
 		</joint>
+		<joint name="${name}_6_joint_torque" type="revolute">
+			<axis xyz="0 0 1"/>
+			<limit lower="${min_damping}" upper="${max_damping}" effort="0" velocity="${rate_daming}" />
+			<safety_controller soft_lower_limit="${min_damping}" soft_upper_limit="${max_damping}" k_position="30" k_velocity="30"/>
+			<parent link="${name}_6_link"/>
+			<child link="${name}_7_link_torque"/>
+		</joint>
 		<link name="${name}_7_link_dummy"/>
 		<link name="${name}_7_link_damping"/>
+		<link name="${name}_7_link_torque"/>
 		<link name="${name}_7_link">
 			<inertial>

Commit message: .

File: kuka_lwr/lwr_description/model/kuka_lwr.urdf.xacro (robot description, xacro)
@@ -63,28 +63,4 @@
       <child link="${name}_1_link"/>
     </joint>
-    <joint name="${name}_0_joint_stiffness" type="revolute">
-      <axis xyz="0 0 1"/>
-      <limit lower="${min_stiffness}" upper="${max_stiffness}" effort="0" velocity="${rate_stiffness}" />
-      <safety_controller soft_lower_limit="${min_stiffness}" soft_upper_limit="${max_stiffness}" k_position="30" k_velocity="30"/>
-      <parent link="${name}_base_link"/>
-      <child link="${name}_1_link_dummy"/>
-    </joint>
-    <joint name="${name}_0_joint_damping" type="revolute">
-      <axis xyz="0 0 1"/>
-      <limit lower="${min_damping}" upper="${max_damping}" effort="0" velocity="${rate_daming}" />
-      <safety_controller soft_lower_limit="${min_damping}" soft_upper_limit="${max_damping}" k_position="30" k_velocity="30"/>
-      <parent link="${name}_base_link"/>
-      <child link="${name}_1_link_damping"/>
-    </joint>
-    <joint name="${name}_0_joint_torque" type="revolute">
-      <axis xyz="0 0 1"/>
-      <limit lower="${-170 * M_PI / 180}" upper="${170 * M_PI / 180}" effort="176" velocity="${velocity_scale * 110 * M_PI / 180}" />
-      <dynamics friction="10.0" damping="1.0"/>
-      <parent link="${name}_base_link"/>
-      <child link="${name}_1_link_torque"/>
-    </joint>
-    <link name="${name}_1_link_dummy"/>
-    <link name="${name}_1_link_damping"/>
-    <link name="${name}_1_link_torque"/>
     <link name="${name}_1_link">
       <inertial>
@@ -129,28 +105,4 @@
       <child link="${name}_2_link"/>
     </joint>
-    <joint name="${name}_1_joint_stiffness" type="revolute">
-      <axis xyz="0 0 1"/>
-      <limit lower="${min_stiffness}" upper="${max_stiffness}" effort="0" velocity="${rate_stiffness}" />
-      <safety_controller soft_lower_limit="${min_stiffness}" soft_upper_limit="${max_stiffness}" k_position="30" k_velocity="30"/>
-      <parent link="${name}_1_link"/>
-      <child link="${name}_2_link_dummy"/>
-    </joint>
-    <joint name="${name}_1_joint_damping" type="revolute">
-      <axis xyz="0 0 1"/>
-      <limit lower="${min_damping}" upper="${max_damping}" effort="0" velocity="${rate_daming}" />
-      <safety_controller soft_lower_limit="${min_damping}" soft_upper_limit="${max_damping}" k_position="30" k_velocity="30"/>
-      <parent link="${name}_1_link"/>
-      <child link="${name}_2_link_damping"/>
-    </joint>
-    <joint name="${name}_1_joint_torque" type="revolute">
-      <axis xyz="0 -1 0"/>
-      <limit lower="${-120 * M_PI / 180}" upper="${120 * M_PI / 180}" effort="176" velocity="${velocity_scale * 110 * M_PI / 180}" />
-      <dynamics friction="10.0" damping="1.0"/>
-      <parent link="${name}_1_link"/>
-      <child link="${name}_2_link_torque"/>
-    </joint>
-    <link name="${name}_2_link_dummy"/>
-    <link name="${name}_2_link_damping"/>
-    <link name="${name}_2_link_torque"/>
     <link name="${name}_2_link">
       <inertial>
@@ -195,28 +147,4 @@
       <child link="${name}_3_link"/>
     </joint>
-    <joint name="${name}_2_joint_stiffness" type="revolute">
-      <axis xyz="0 0 1"/>
-      <limit lower="${min_stiffness}" upper="${max_stiffness}" effort="0" velocity="${rate_stiffness}" />
-      <safety_controller soft_lower_limit="${min_stiffness}" soft_upper_limit="${max_stiffness}" k_position="30" k_velocity="30"/>
-      <parent link="${name}_2_link"/>
-      <child link="${name}_3_link_dummy"/>
-    </joint>
-    <joint name="${name}_2_joint_damping" type="revolute">
-      <axis xyz="0 0 1"/>
-      <limit lower="${min_damping}" upper="${max_damping}" effort="0" velocity="${rate_daming}" />
-      <safety_controller soft_lower_limit="${min_damping}" soft_upper_limit="${max_damping}" k_position="30" k_velocity="30"/>
-      <parent link="${name}_2_link"/>
-      <child link="${name}_3_link_damping"/>
-    </joint>
-    <joint name="${name}_2_joint_torque" type="revolute">
-      <axis xyz="0 0 1"/>
-      <limit lower="${min_stiffness}" upper="${max_stiffness}" effort="0" velocity="${rate_stiffness}" />
-      <safety_controller soft_lower_limit="${min_stiffness}" soft_upper_limit="${max_stiffness}" k_position="30" k_velocity="30"/>
-      <parent link="${name}_2_link"/>
-      <child link="${name}_3_link_torque"/>
-    </joint>
-    <link name="${name}_3_link_dummy"/>
-    <link name="${name}_3_link_damping"/>
-    <link name="${name}_3_link_torque"/>
     <link name="${name}_3_link">
       <inertial>
@@ -261,28 +189,4 @@
       <child link="${name}_4_link"/>
     </joint>
-    <joint name="${name}_3_joint_stiffness" type="revolute">
-      <axis xyz="0 0 1"/>
-      <limit lower="${min_stiffness}" upper="${max_stiffness}" effort="0" velocity="${rate_stiffness}" />
-      <safety_controller soft_lower_limit="${min_stiffness}" soft_upper_limit="${max_stiffness}" k_position="30" k_velocity="30"/>
-      <parent link="${name}_3_link"/>
-      <child link="${name}_4_link_dummy"/>
-    </joint>
-    <joint name="${name}_3_joint_damping" type="revolute">
-      <axis xyz="0 0 1"/>
-      <limit lower="${min_damping}" upper="${max_damping}" effort="0" velocity="${rate_daming}" />
-      <safety_controller soft_lower_limit="${min_damping}" soft_upper_limit="${max_damping}" k_position="30" k_velocity="30"/>
-      <parent link="${name}_3_link"/>
-      <child link="${name}_4_link_damping"/>
-    </joint>
-    <joint name="${name}_3_joint_torque" type="revolute">
-      <axis xyz="0 1 0"/>
-      <limit lower="${-120 * M_PI / 180}" upper="${120 * M_PI / 180}" effort="100" velocity="${velocity_scale * 128 * M_PI / 180}" />
-      <dynamics friction="10.0" damping="1.0"/>
-      <parent link="${name}_3_link"/>
-      <child link="${name}_4_link_torque"/>
-    </joint>
-    <link name="${name}_4_link_dummy"/>
-    <link name="${name}_4_link_damping"/>
-    <link name="${name}_4_link_torque"/>
     <link name="${name}_4_link">
       <inertial>
@@ -327,28 +231,4 @@
       <child link="${name}_5_link"/>
     </joint>
-    <joint name="${name}_4_joint_stiffness" type="revolute">
-      <axis xyz="0 0 1"/>
-      <limit lower="${min_stiffness}" upper="${max_stiffness}" effort="0" velocity="${rate_stiffness}" />
-      <safety_controller soft_lower_limit="${min_stiffness}" soft_upper_limit="${max_stiffness}" k_position="30" k_velocity="30"/>
-      <parent link="${name}_4_link"/>
-      <child link="${name}_5_link_dummy"/>
-    </joint>
-    <joint name="${name}_4_joint_damping" type="revolute">
-      <axis xyz="0 0 1"/>
-      <limit lower="${min_damping}" upper="${max_damping}" effort="0" velocity="${rate_daming}" />
-      <safety_controller soft_lower_limit="${min_damping}" soft_upper_limit="${max_damping}" k_position="30" k_velocity="30"/>
-      <parent link="${name}_4_link"/>
-      <child link="${name}_5_link_damping"/>
-    </joint>
-    <joint name="${name}_4_joint_torque" type="revolute">
-      <axis xyz="0 0 1"/>
-      <limit lower="${min_damping}" upper="${max_damping}" effort="0" velocity="${rate_daming}" />
-      <safety_controller soft_lower_limit="${min_damping}" soft_upper_limit="${max_damping}" k_position="30" k_velocity="30"/>
-      <parent link="${name}_4_link"/>
-      <child link="${name}_5_link_torque"/>
-    </joint>
-    <link name="${name}_5_link_dummy"/>
-    <link name="${name}_5_link_damping"/>
-    <link name="${name}_5_link_torque"/>
     <link name="${name}_5_link">
       <inertial>
@@ -393,28 +273,4 @@
       <child link="${name}_6_link"/>
     </joint>
-    <joint name="${name}_5_joint_stiffness" type="revolute">
-      <axis xyz="0 0 1"/>
-      <limit lower="${min_stiffness}" upper="${max_stiffness}" effort="0" velocity="${rate_stiffness}" />
-      <safety_controller soft_lower_limit="${min_stiffness}" soft_upper_limit="${max_stiffness}" k_position="30" k_velocity="30"/>
-      <parent link="${name}_5_link"/>
-      <child link="${name}_6_link_dummy"/>
-    </joint>
-    <joint name="${name}_5_joint_damping" type="revolute">
-      <axis xyz="0 0 1"/>
-      <limit lower="${min_damping}" upper="${max_damping}" effort="0" velocity="${rate_daming}" />
-      <safety_controller soft_lower_limit="${min_damping}" soft_upper_limit="${max_damping}" k_position="30" k_velocity="30"/>
-      <parent link="${name}_5_link"/>
-      <child link="${name}_6_link_damping"/>
-    </joint>
-    <joint name="${name}_5_joint_torque" type="revolute">
-      <axis xyz="0 0 1"/>
-      <limit lower="${min_damping}" upper="${max_damping}" effort="0" velocity="${rate_daming}" />
-      <safety_controller soft_lower_limit="${min_damping}" soft_upper_limit="${max_damping}" k_position="30" k_velocity="30"/>
-      <parent link="${name}_5_link"/>
-      <child link="${name}_6_link_torque"/>
-    </joint>
-    <link name="${name}_6_link_dummy"/>
-    <link name="${name}_6_link_damping"/>
-    <link name="${name}_6_link_torque"/>
     <link name="${name}_6_link">
       <inertial>
@@ -446,28 +302,4 @@
       <child link="${name}_7_link"/>
     </joint>
-    <joint name="${name}_6_joint_stiffness" type="revolute">
-      <axis xyz="0 0 1"/>
-      <limit lower="${min_stiffness}" upper="${max_stiffness}" effort="0" velocity="${rate_stiffness}" />
-      <safety_controller soft_lower_limit="${min_stiffness}" soft_upper_limit="${max_stiffness}" k_position="30" k_velocity="30"/>
-      <parent link="${name}_6_link"/>
-      <child link="${name}_7_link_dummy"/>
-    </joint>
-    <joint name="${name}_6_joint_damping" type="revolute">
-      <axis xyz="0 0 1"/>
-      <limit lower="${min_damping}" upper="${max_damping}" effort="0" velocity="${rate_daming}" />
-      <safety_controller soft_lower_limit="${min_damping}" soft_upper_limit="${max_damping}" k_position="30" k_velocity="30"/>
-      <parent link="${name}_6_link"/>
-      <child link="${name}_7_link_damping"/>
-    </joint>
-    <joint name="${name}_6_joint_torque" type="revolute">
-      <axis xyz="0 0 1"/>
-      <limit lower="${min_damping}" upper="${max_damping}" effort="0" velocity="${rate_daming}" />
-      <safety_controller soft_lower_limit="${min_damping}" soft_upper_limit="${max_damping}" k_position="30" k_velocity="30"/>
-      <parent link="${name}_6_link"/>
-      <child link="${name}_7_link_torque"/>
-    </joint>
-    <link name="${name}_7_link_dummy"/>
-    <link name="${name}_7_link_damping"/>
-    <link name="${name}_7_link_torque"/>
     <link name="${name}_7_link">
       <inertial>
