Commit message: Much simpler solution; xacro arguments can have default values.

File: kuka_lwr/lwr_description/model/kuka_lwr.urdf.xacro (robot description, xacro)
@@ -1,16 +1,334 @@
 <?xml version="1.0"?>
 <robot name="kuka_lwr" xmlns:xacro="http://www.ros.org/wiki/xacro">
-  <xacro:include filename="$(find lwr_description)/model/kuka_lwr_robot.urdf.xacro"/>
-  <!-- This is a model of the KUKA LWR that is rooted in the 'world' frame. -->
-  <xacro:macro name="kuka_lwr" params="name *origin">
-    <link name="world"/>
-    <gazebo reference="world">
+  <!-- utils /-->
+  <xacro:include filename="$(find lwr_description)/model/utils.xacro"/>
+  <xacro:include filename="$(find lwr_description)/model/kuka_materials.xacro"
+	         />
+  <!-- gazebo and transmission models /-->
+  <xacro:include filename="$(find lwr_description)/model/kuka_lwr.gazebo.xacro"/>
+  <xacro:include filename="$(find lwr_description)/model/kuka_lwr.transmission.xacro"/>
+  <!-- properties /-->
+  <xacro:property name="base_mass" value="2.0"/>
+  <xacro:property name="link_mass" value="2.0"/>
+  <xacro:property name="velocity_scale" value="1"/>
+  <xacro:property name="effort_scale" value="1"/>
+  <xacro:property name="max_stiffness" value="5000"/>
+  <xacro:property name="min_stiffness" value="0"/>
+  <xacro:property name="rate_stiffness" value="20000"/> <!-- reflex to stiffness -->
+  <xacro:property name="max_damping" value="500"/>
+  <xacro:property name="min_damping" value="0"/>
+  <xacro:property name="rate_daming" value="20000"/>
+  <!-- URDF model with default base_link (world)-->
+  <xacro:macro name="kuka_lwr" params="name base_link:=world *origin">
+    <link name="${base_link}"/>
+    <gazebo reference="${base_link}">
       <static>true</static>
       <turnGravityOff>true</turnGravityOff>
     </gazebo>
-    <xacro:kuka_lwr_variable_root name="${name}"
-                                  base_link="world"
-                                  >
-    </xacro:kuka_lwr_variable_root>
+    <!-- First (shoulder) element of the arm. Fixed to its parent. -->
+    <joint name="${name}_base_joint" type="fixed">
+      <insert_block name="origin"/>
+      <origin xyz="0 0 0" rpy="0 0 0"/>
+      <parent link="${base_link}"/>
+      <child link="${name}_base_link"/>
+    </joint>
+    <link name="${name}_base_link">
+      <inertial>
+	<mass value="${base_mass}"/>
+	<origin xyz="0 0 0.055"  />
+	<cylinder_inertia_def radius="0.06" length="0.11" mass="${base_mass}"/>
+      </inertial>
+      <visual>
+	<origin xyz="0 0 0" rpy="0 0 ${M_PI}"/>
+	<geometry>
+            <mesh filename="package://lwr_description/meshes_arm/arm_base.dae"/>
+	</geometry>
+	<material name="Kuka/Orange"/>
+      </visual>
+      <collision>
+	<origin xyz="0 0 0.055" rpy="0 0 ${M_PI}"/>
+	<geometry>
+	  <!-- <mesh filename="package://lwr_description/meshes/convex/arm_base_convex.stl"/> -->
+	  <cylinder radius="0.07" length="0.11"/>
+	</geometry>
+      </collision>
+    </link>
+    <!-- Second segment of the arm. Joint along z-axis -->
+    <joint name="${name}_0_joint" type="revolute">
+      <origin xyz="0 0 0.11" rpy="0 0 0"/>
+      <axis xyz="0 0 1"/>
+      <limit lower="${-170 * M_PI / 180}" upper="${170 * M_PI / 180}" effort="176" velocity="${velocity_scale * 110 * M_PI / 180}" />
+      <dynamics friction="10.0" damping="1.0"/>
+      <parent link="${name}_base_link"/>
+      <child link="${name}_1_link"/>
+    </joint>
+<!-- 			LINK 1 			-->
+    <link name="${name}_1_link">
+      <inertial>
+	<mass value="${link_mass}"/>
+	<origin rpy="0 0 0" xyz="0 -0.06 0.130"/>
+	<cuboid_inertia_def length="0.12" width="0.06" height="0.260" mass="${link_mass}"/>
+      </inertial>
+      <visual>
+            <origin xyz="0 0 0" rpy="0 0 ${M_PI}"/>
+            <geometry>
+              <mesh filename="package://lwr_description/meshes_arm/arm_segment_a.dae"/>
+            </geometry>
+            <material name="Orange"/>
+      </visual>
+      <collision>
+	<origin xyz="0 0 0.0" rpy="0 0 0"/>
+	<geometry>
+	  <!--mesh filename="package://lwr_description/meshes/convex/arm_segment_a_convex.stl"/-->
+	  <sphere radius="0.07"/>
+	</geometry>
+      </collision>
+      <collision>
+	<origin xyz="0 0.06 0.2" rpy="0 0 0"/>
+	<geometry>
+	  <sphere radius="0.07"/>
+	</geometry>
+      </collision>
+      <collision>
+	<origin xyz="0 0.03 0.1" rpy="-0.291 0 0"/>
+	<geometry>
+	  <cylinder radius="0.07" length="0.208"/>
+	</geometry>
+      </collision>
+    </link>
+    <!-- Third segment of the arm. Joint along y-axis -->
+    <joint name="${name}_1_joint" type="revolute">
+      <origin xyz="0 0 0.2005" rpy="0 0 0"/>
+      <axis xyz="0 -1 0"/>
+      <limit lower="${-120 * M_PI / 180}" upper="${120 * M_PI / 180}" effort="176" velocity="${velocity_scale * 110 * M_PI / 180}" />
+      <dynamics friction="10.0" damping="1.0"/>
+      <parent link="${name}_1_link"/>
+      <child link="${name}_2_link"/>
+    </joint>
+<!-- 			LINK 2 			-->
+    <link name="${name}_2_link">
+      <inertial>
+	<mass value="${link_mass}"/>
+	<origin rpy="0 0 0" xyz="0 0.06 ${0.130 - 0.06}"/>
+	<cuboid_inertia_def length="0.12" width="0.06" height="0.260" mass="${link_mass}"/>
+      </inertial>
+        <visual>
+          <origin xyz="0 0 0.2" rpy="${M_PI} 0 ${M_PI}"/>
+          <geometry>
+            <mesh filename="package://lwr_description/meshes_arm/arm_segment_b.dae"/>
+          </geometry>
+          <material name="Orange"/>
+        </visual>
+      <collision>
+	<origin xyz="0 0 0.2" rpy="0 0 0"/>
+	<geometry>
+	  <!--mesh filename="package://lwr_description/meshes/convex/arm_segment_b_convex.stl"/-->
+	  <sphere radius="0.07"/>
+	</geometry>
+      </collision>
+      <collision>
+	<origin xyz="0 -0.06 0.0" rpy="0 0 0"/>
+	<geometry>
+	  <sphere radius="0.07"/>
+	</geometry>
+      </collision>
+      <collision>
+	<origin xyz="0 -0.03 0.1" rpy="-0.291 0 0"/>
+	<geometry>
+	  <cylinder radius="0.07" length="0.208"/>
+	</geometry>
+      </collision>
+    </link>
+    <!-- Fourth element of the arm. z-axis -->
+    <joint name="${name}_2_joint" type="revolute">
+      <origin xyz="0 0 0.20" rpy="0 0 0"/>
+      <axis xyz="0 0 1"/>
+      <limit lower="${-170 * M_PI / 180}" upper="${170 * M_PI / 180}" effort="100" velocity="${velocity_scale * 128 * M_PI / 180}" />
+      <dynamics friction="10.0" damping="1.0"/>
+      <parent link="${name}_2_link"/>
+      <child link="${name}_3_link"/>
+    </joint>
+<!-- 			LINK 3 			-->
+    <link name="${name}_3_link">
+      <inertial>
+	<mass value="${link_mass}"/>
+	<origin rpy="0 0 0" xyz="0 0.06 0.130"/>
+	<cuboid_inertia_def length="0.12" width="0.06" height="0.260" mass="${link_mass}"/>
+      </inertial>
+      <visual>
+       <origin xyz="0 0 0" rpy="0 0 0"/>
+       <geometry>
+       	 <mesh filename="package://lwr_description/meshes_arm/arm_segment_a.dae"/>
+        </geometry>
+        <material name="Orange"/>
+      </visual>
+      <collision>
+	<origin xyz="0 0 0.0" rpy="0 0 0"/>
+	<geometry>
+	  <!--mesh filename="package://lwr_description/meshes/convex/arm_segment_a_convex.stl"/-->
+	  <sphere radius="0.07"/>
+	</geometry>
+      </collision>
+      <collision>
+	<origin xyz="0 -0.06 0.2" rpy="0 0 0"/>
+	<geometry>
+	  <sphere radius="0.07"/>
+	</geometry>
+      </collision>
+      <collision>
+	<origin xyz="0 -0.03 0.1" rpy="0.291 0 0"/>
+	<geometry>
+	  <cylinder radius="0.07" length="0.208"/>
+	</geometry>
+      </collision>
+    </link>
+    <!-- fifth element of the arm. x-axis -->
+    <joint name="${name}_3_joint" type="revolute">
+      <origin xyz="0 0 0.20" rpy="0 0 0"/>
+      <axis xyz="0 1 0"/>
+      <limit lower="${-120 * M_PI / 180}" upper="${120 * M_PI / 180}" effort="100" velocity="${velocity_scale * 128 * M_PI / 180}" />
+      <dynamics friction="10.0" damping="1.0"/>
+      <parent link="${name}_3_link"/>
+      <child link="${name}_4_link"/>
+    </joint>
+<!-- 			LINK 4 			-->
+    <link name="${name}_4_link">
+      <inertial>
+	<mass value="${link_mass}"/>
+	<origin rpy="0 0 0" xyz="0 -0.06 ${0.130 - 0.06}"/>
+	<cuboid_inertia_def length="0.12" width="0.06" height="0.2600" mass="${link_mass}"/>
+      </inertial>
+      <visual>
+        <origin xyz="0 0 0.2" rpy="0 ${M_PI} ${M_PI}"/>
+         <geometry>
+            <mesh filename="package://lwr_description/meshes_arm/arm_segment_b.dae"/>
+      	 </geometry>
+      	<material name="Orange"/>
+      </visual>
+      <collision>
+	<origin xyz="0 0 0.2" rpy="0 0 0"/>
+	<geometry>
+	  <!--mesh filename="package://lwr_description/meshes/convex/arm_segment_b_convex.stl"/-->
+	  <sphere radius="0.07"/>
+	</geometry>
+      </collision>
+      <collision>
+	<origin xyz="0 0.06 0.0" rpy="0 0 0"/>
+	<geometry>
+	  <sphere radius="0.07"/>
+	</geometry>
+      </collision>
+      <collision>
+	<origin xyz="0 0.03 0.1" rpy="0.291 0 0"/>
+	<geometry>
+	  <cylinder radius="0.07" length="0.208"/>
+	</geometry>
+      </collision>
+    </link>
+    <!-- Sixth element of the arm. z-axis -->
+    <joint name="${name}_4_joint" type="revolute">
+      <origin xyz="0 0 0.20" rpy="0 0 0"/>
+      <axis xyz="0 0 1"/>
+      <limit lower="${-170 * M_PI / 180}" upper="${170 * M_PI / 180}" effort="100" velocity="${velocity_scale * 204 * M_PI / 180}" />
+      <dynamics friction="10.0" damping="1.0"/>
+      <parent link="${name}_4_link"/>
+      <child link="${name}_5_link"/>
+    </joint>
+<!-- 			LINK 5 			-->
+    <link name="${name}_5_link">
+      <inertial>
+	<mass value="${link_mass}"/>
+	<origin rpy="0 0 0" xyz="0 0 0.124"/>
+	<cuboid_inertia_def length="0.12" width="0.06" height="0.248" mass="${link_mass}"/>
+      </inertial>
+      <visual>
+      	<origin xyz="0 0 0" rpy="0 0 ${M_PI}"/>
+      	  <geometry name="${name}_arm_5_geom">
+             <mesh filename="package://lwr_description/meshes_arm/arm_segment_last.dae"/>
+           </geometry>
+         <material name="Orange"/>
+      </visual>
+      <collision>
+	<origin xyz="0 0 0.0" rpy="0 0 0"/>
+	<geometry>
+	  <!--mesh filename="package://lwr_description/meshes/convex/arm_segment_last_convex.stl"/-->
+	  <sphere radius="0.07"/>
+	</geometry>
+      </collision>
+      <collision>
+	<origin xyz="0 0.04 0.19" rpy="0 0 0"/>
+	<geometry>
+	  <sphere radius="0.07"/>
+	</geometry>
+      </collision>
+      <collision>
+	<origin xyz="0 0.02 0.095" rpy="-0.207 0 0"/>
+	<geometry>
+	  <cylinder radius="0.07" length="0.198"/>
+	</geometry>
+      </collision>
+    </link>
+    <!-- Seventh element of the arm. z-axis -->
+    <joint name="${name}_5_joint" type="revolute">
+      <origin xyz="0 0 0.19" rpy="0 0 0"/>
+      <axis xyz="0 -1 0"/>
+      <limit lower="${-120 * M_PI / 180}" upper="${120 * M_PI / 180}" effort="38" velocity="${velocity_scale * 184 * M_PI / 180}" />
+      <dynamics friction="10.0" damping="1.0"/>
+      <parent link="${name}_5_link"/>
+      <child link="${name}_6_link"/>
+    </joint>
+<!-- 			LINK 6 			-->
+    <link name="${name}_6_link">
+      <inertial>
+	<mass value="0.2"/>
+	<origin rpy="0 0 0" xyz="0 0 0.0625"/>
+	<cuboid_inertia_def length="0.125" width="0.125" height="0.125" mass="0.2"/>
+      </inertial>
+      <visual>
+      	<origin xyz="0 0 0" rpy="0 0 ${M_PI}"/>
+        <geometry>
+      	  <mesh filename="package://lwr_description/meshes_arm/arm_wrist.dae"/>
+         </geometry>
+         <material name="Grey"/>
+      </visual>
+      <collision>
+	<origin xyz="0 0 0" rpy="0 0 ${M_PI}"/>
+	<geometry>
+	  <mesh filename="package://lwr_description/meshes/convex/arm_wrist_convex.stl"/>
+	</geometry>
+      </collision>
+    </link>
+    <!-- Eighth element of the arm. z-axis -->
+    <joint name="${name}_6_joint" type="revolute">
+      <origin xyz="0 0 0.078" rpy="0 0 0"/>
+      <axis xyz="0 0 1"/>
+      <limit lower="${-170 * M_PI / 180}" upper="${170 * M_PI / 180}" effort="38" velocity="${velocity_scale * 184 * M_PI / 180}" />
+      <dynamics friction="10.0" damping="1.0"/>
+      <parent link="${name}_6_link"/>
+      <child link="${name}_7_link"/>
+    </joint>
+<!-- 			LINK 7 			-->
+    <link name="${name}_7_link">
+      <inertial>
+	<mass value="0.2"/>
+	<origin xyz="0 0 0"/>
+	<cuboid_inertia_def length="1" width="1" height="1" mass="0.2"/>
+      </inertial>
+      <visual>
+	<origin xyz="0 0 0" rpy="0 0 ${M_PI}"/>
+	<geometry>
+	  <mesh filename="package://lwr_description/meshes/link_7.dae"/>
+	</geometry>
+	<material name="Kuka/DarkGrey"/>
+      </visual>
+      <collision>
+	<origin xyz="0 0 0" rpy="0 0 ${M_PI}"/>
+	<geometry>
+	  <cylinder radius="0.04" length="0.05"/>
+	</geometry>
+      </collision>
+    </link>
+    <xacro:kuka_lwr_gazebo name="${name}"/>
+    <xacro:kuka_lwr_transmission name="${name}"/>
   </xacro:macro>
 </robot>

Commit message: Add changes to be able to work with two robots at the same time

File: kuka_lwr/lwr_description/model/kuka_lwr.urdf.xacro (robot description, xacro)
@@ -20,5 +20,5 @@
   <xacro:property name="rate_daming" value="20000"/>
   <!-- URDF model with default base_link (world)-->
-  <xacro:macro name="kuka_lwr" params="name base_link:=world *origin">
+  <xacro:macro name="kuka_lwr" params="name base_link:=world_2 *origin">
     <link name="${base_link}"/>
     <gazebo reference="${base_link}">

Commit message: Fix simulation launch file and kuka_lwr urdf xacro file

File: kuka_lwr/lwr_description/model/kuka_lwr.urdf.xacro (robot description, xacro)
@@ -35,7 +35,7 @@
     <link name="${name}_base_link">
       <inertial>
-	<mass value="${base_mass}"/>
-	<origin xyz="0 0 0.055"  />
-	<cylinder_inertia_def radius="0.06" length="0.11" mass="${base_mass}"/>
+	      <mass value="${base_mass}"/>
+	      <origin xyz="0 0 0.055"  />
+	      <xacro:cylinder_inertia_def radius="0.06" length="0.11" mass="${base_mass}"/>
       </inertial>
       <visual>
@@ -68,5 +68,5 @@
 	<mass value="${link_mass}"/>
 	<origin rpy="0 0 0" xyz="0 -0.06 0.130"/>
-	<cuboid_inertia_def length="0.12" width="0.06" height="0.260" mass="${link_mass}"/>
+	<xacro:cuboid_inertia_def length="0.12" width="0.06" height="0.260" mass="${link_mass}"/>
       </inertial>
       <visual>
@@ -111,5 +111,5 @@
 	<mass value="${link_mass}"/>
 	<origin rpy="0 0 0" xyz="0 0.06 ${0.130 - 0.06}"/>
-	<cuboid_inertia_def length="0.12" width="0.06" height="0.260" mass="${link_mass}"/>
+	<xacro:cuboid_inertia_def length="0.12" width="0.06" height="0.260" mass="${link_mass}"/>
       </inertial>
         <visual>
@@ -154,5 +154,5 @@
 	<mass value="${link_mass}"/>
 	<origin rpy="0 0 0" xyz="0 0.06 0.130"/>
-	<cuboid_inertia_def length="0.12" width="0.06" height="0.260" mass="${link_mass}"/>
+	<xacro:cuboid_inertia_def length="0.12" width="0.06" height="0.260" mass="${link_mass}"/>
       </inertial>
       <visual>
@@ -197,5 +197,5 @@
 	<mass value="${link_mass}"/>
 	<origin rpy="0 0 0" xyz="0 -0.06 ${0.130 - 0.06}"/>
-	<cuboid_inertia_def length="0.12" width="0.06" height="0.2600" mass="${link_mass}"/>
+	<xacro:cuboid_inertia_def length="0.12" width="0.06" height="0.2600" mass="${link_mass}"/>
       </inertial>
       <visual>
@@ -240,5 +240,5 @@
 	<mass value="${link_mass}"/>
 	<origin rpy="0 0 0" xyz="0 0 0.124"/>
-	<cuboid_inertia_def length="0.12" width="0.06" height="0.248" mass="${link_mass}"/>
+	<xacro:cuboid_inertia_def length="0.12" width="0.06" height="0.248" mass="${link_mass}"/>
       </inertial>
       <visual>
@@ -283,5 +283,5 @@
 	<mass value="0.2"/>
 	<origin rpy="0 0 0" xyz="0 0 0.0625"/>
-	<cuboid_inertia_def length="0.125" width="0.125" height="0.125" mass="0.2"/>
+	<xacro:cuboid_inertia_def length="0.125" width="0.125" height="0.125" mass="0.2"/>
       </inertial>
       <visual>
@@ -313,5 +313,5 @@
 	<mass value="0.2"/>
 	<origin xyz="0 0 0"/>
-	<cuboid_inertia_def length="1" width="1" height="1" mass="0.2"/>
+	<xacro:cuboid_inertia_def length="1" width="1" height="1" mass="0.2"/>
       </inertial>
       <visual>
